Commit message: update

File: description/robot_core.xacro (robot description, xacro)
@@ -1,15 +1,15 @@
 <?xml version="1.0"?>
 <robot xmlns:xacro="http://www.ros.org/wiki/xacro"  name="robot">
-    <material name="write">
+    <material name="white">
       <color rgba="1 1 1 1"/>
     </material>
     <material name="orange">
-      <color rgba="1 1 1 1"/>
+      <color rgba="1 0.3 0.1 1"/>
     </material>
     <material name="blue">
-      <color rgba="1 1 1 1"/>
+      <color rgba="0.2 0.2 1 1"/>
     </material>
     <material name="black">
-      <color rgba="1 1 1 1"/>
+      <color rgba="0 0 0 1"/>
     </material>
     <link name="base_link">
@@ -18,9 +18,9 @@
        <parent link="base_link"/>
        <child link="chassis"/>
-       <origin xyz="0.1 0 0 "/>
+       <origin xyz="-0.1 0 0 "/>
     </joint>
     <link name="chassis">
        <visual>
-           <origin xyz="0.15 0.15 0.075"/>
+           <origin xyz="0.15 0 0.075"/>
            <geometry>
                <box size= "0.3 0.3 0.15"/>

Commit message: ep2

File: description/robot_core.xacro (robot description, xacro)
@@ -13,6 +13,8 @@
       <color rgba="0 0 0 1"/>
     </material>
+    <!-- base link -->
     <link name="base_link">
     </link>
+    <!-- chassis link -->
     <joint name="chassis_joint" type="fixed">
        <parent link="base_link"/>
@@ -29,3 +31,35 @@
        </visual>
     </link>
+    <!-- left whelel link -->
+    <joint name="left_wheel_joint" type="continuous">
+       <parent link="base_link"/>
+       <child link="left_wheel"/>
+       <origin xyz="0 0.175 0 " rpy="-${pi/2} 0 0 "/>
+       <axis xyz="0 0 1" />
+    </joint>
+    <link name="left_wheel">
+       <visual>
+           <origin xyz="0.15 0 0.075"/>
+           <geometry>
+               <cylinder radius= "0.05" length="0.04"/>
+           </geometry>
+           <material name="blue"/>
+       </visual>
+    </link>
+    <!-- right whelel link -->
+    <joint name="right_wheel_joint" type="continuous">
+       <parent link="base_link"/>
+       <child link="right_wheel"/>
+       <origin xyz="0 -0.175 0 " rpy="${pi/2} 0 0 "/>
+       <axis xyz="0 0 -1" />
+    </joint>
+    <link name="right_wheel">
+       <visual>
+           <origin xyz="0.15 0 0.075"/>
+           <geometry>
+               <cylinder radius= "0.05" lenght="0.04"/>
+           </geometry>
+           <material name="blue"/>
+       </visual>
+    </link>
 </robot>

Commit message: create uidf

File: description/robot_core.xacro (robot description, xacro)
@@ -1,6 +1,7 @@
 <?xml version="1.0"?>
 <robot xmlns:xacro="http://www.ros.org/wiki/xacro"  name="robot">
+    <xacro:include filename="inertial_macros.xacro"/>
     <material name="white">
-      <color rgba="0.1 1 1 1"/>
+      <color rgba="1 1 1 1"/>
     </material>
     <material name="orange">
@@ -30,6 +31,16 @@
            <material name="white"/>
        </visual>
+       <collision>
+           <origin xyz="0.15 0 0.075"/>
+           <geometry>
+               <box size= "0.3 0.3 0.15"/>
+           </geometry>
+           <material name="white"/>
+       </collision>
+       <xacro:inertial_box mass="0.5" x="0.3" y="0.3" z="0.15">
+         <origin xyz="0.15 0 0.075" rpy="0 0 0"/>
+        </xacro:inertial_box>
     </link>
-    <!-- left whelel link -->
+    <!-- left whelel link back-->
     <joint name="left_wheel_joint" type="continuous">
        <parent link="base_link"/>
@@ -40,5 +51,4 @@
     <link name="left_wheel">
        <visual>
-           <origin xyz="0.15 0 0.075"/>
            <geometry>
                <cylinder radius= "0.05" length="0.04"/>
@@ -46,6 +56,15 @@
            <material name="blue"/>
        </visual>
+       <collision>
+           <geometry>
+               <cylinder radius= "0.05" length="0.04"/>
+           </geometry>
+           <material name="blue"/>
+       </collision>
+       <xacro:inertial_cylinder mass="0.1" length="0.04" radius="0.05" >
+         <origin xyz="0 0 0" rpy="0 0 0"/>
+       </xacro:inertial_cylinder>
     </link>
-    <!-- right whelel link -->
+    <!-- right whelel link back -->
     <joint name="right_wheel_joint" type="continuous">
        <parent link="base_link"/>
@@ -56,10 +75,66 @@
     <link name="right_wheel">
        <visual>
-           <origin xyz="0.15 0 0.075"/>
            <geometry>
-               <cylinder radius= "0.05" lenght="0.04"/>
+               <cylinder radius= "0.05" length="0.04"/>
            </geometry>
            <material name="blue"/>
        </visual>
+       <collision>
+           <geometry>
+               <cylinder radius= "0.05" length="0.04"/>
+           </geometry>
+           <material name="blue"/>
+       </collision>
+       <xacro:inertial_cylinder mass="0.1" length="0.04" radius="0.05" >
+         <origin xyz="0 0 0" rpy="0 0 0"/>
+        </xacro:inertial_cylinder>
+    </link>
+    <!-- left whelel link forward-->
+    <joint name="left_wheel_joint_forward" type="continuous">
+       <parent link="base_link"/>
+       <child link="left_wheel_forward"/>
+       <origin xyz="0.15 0.175 0 " rpy="-${pi/2} 0 0 "/>
+       <axis xyz="0 0 1" />
+    </joint>
+    <link name="left_wheel_forward">
+       <visual>
+           <geometry>
+               <cylinder radius= "0.05" length="0.04"/>
+           </geometry>
+           <material name="blue"/>
+       </visual>
+       <collision>
+           <geometry>
+               <cylinder radius= "0.05" length="0.04"/>
+           </geometry>
+           <material name="blue"/>
+       </collision>
+       <xacro:inertial_cylinder mass="0.1" length="0.04" radius="0.05" >
+         <origin xyz="0 0 0" rpy="0 0 0"/>
+        </xacro:inertial_cylinder>
+    </link>
+    <!-- right whelel link forward -->
+    <joint name="right_wheel_joint_forward" type="continuous">
+       <parent link="base_link"/>
+       <child link="right_wheel_forward"/>
+       <origin xyz="0.15 -0.175 0 " rpy="${pi/2} 0 0 "/>
+       <axis xyz="0 0 -1" />
+    </joint>
+    <link name="right_wheel_forward">
+       <visual>
+           <geometry>
+               <cylinder radius= "0.05" length="0.04"/>
+           </geometry>
+           <material name="blue"/>
+       </visual>
+      <collision>
+           <geometry>
+               <cylinder radius= "0.05" length="0.04"/>
+           </geometry>
+           <material name="blue"/>
+       </collision>
+       <xacro:inertial_cylinder mass="0.1" length="0.04" radius="0.05" >
+         <origin xyz="0 0 0" rpy="0 0 0"/>
+        </xacro:inertial_cylinder>
     </link>
 </robot>

Commit message: Driving robot virtual robot

File: description/robot_core.xacro (robot description, xacro)
@@ -42,4 +42,7 @@
         </xacro:inertial_box>
     </link>
+    <gazebo reference="chassis">
+    <material>Gazebo/White</material>
+    </gazebo>
     <!-- left whelel link back-->
     <joint name="left_wheel_joint" type="continuous">
@@ -66,4 +69,7 @@
        </xacro:inertial_cylinder>
     </link>
+           <gazebo reference="left_wheel">
+    <material>Gazebo/Blue</material>
+    </gazebo>
     <!-- right whelel link back -->
     <joint name="right_wheel_joint" type="continuous">
@@ -90,4 +96,7 @@
         </xacro:inertial_cylinder>
     </link>
+               <gazebo reference="right_wheel">
+    <material>Gazebo/Blue</material>
+    </gazebo>
     <!-- left whelel link forward-->
     <joint name="left_wheel_joint_forward" type="continuous">
@@ -114,4 +123,7 @@
         </xacro:inertial_cylinder>
     </link>
+                   <gazebo reference="left_wheel_forward">
+    <material>Gazebo/Blue</material>
+    </gazebo>
     <!-- right whelel link forward -->
     <joint name="right_wheel_joint_forward" type="continuous">
@@ -138,3 +150,6 @@
         </xacro:inertial_cylinder>
     </link>
+        <gazebo reference="right_wheel_forward">
+    <material>Gazebo/Blue</material>
+    </gazebo>
 </robot>

Commit message: clip9 not finish camera.xacro

File: description/robot_core.xacro (robot description, xacro)
@@ -13,4 +13,7 @@
     <material name="black">
       <color rgba="0 0 0 1"/>
+    </material>
+    <material name="red">
+      <color rgba="1 0 0 1"/>
     </material>
     <!-- base link -->
