Commit message: last vm

File: description/depth_camera.xacro (robot description, xacro)
@@ -22,5 +22,5 @@
     <gazebo reference="camera_link">
         <material>Gazebo/Red</material>
-      <sensor name="camera" type="camera">
+      <sensor name="camera" type="depth">
               <pose> 0 0 0 0 0 0 </pose>
             <visualize>true</visualize>
@@ -40,4 +40,6 @@
             <plugin name="camera_controller" filename="libgazebo_ros_camera.so">
                 <frame_name>camera_link_optical</frame_name>
+                <min_depth>0.1</min_depth>
+                <max_depth>100.0</max_depth>
             </plugin>
         </sensor>

File: description/lidar.xacro (robot description, xacro)
@@ -11,5 +11,5 @@
                <cylinder radius= "0.05" length="0.04"/>
            </geometry>
-           <material name="red"/>
+           <material name="blue"/>
        </visual>
        <collision>
@@ -27,5 +27,5 @@
         <sensor name="laser" type="ray">
             <pose> 0 0 0 0 0 0 </pose>
-            <visualize>true</visualize>
+            <visualize>false</visualize>
             <update_rate>10</update_rate>
             <ray>
@@ -44,6 +44,8 @@
             <plugin name="laser_controller" filename="libgazebo_ros_ray_sensor.so">
                 <ros>
-                    <argument>~/out:=scan</argument>
+                    <argument>--remap ~/out:=scan</argument>
+                    <!-- it telling it what topic to publish it onto   -->
                 </ros>
+                 <!-- publish laserscan msg to scan -->
                 <output_type>sensor_msgs/LaserScan</output_type>
                 <frame_name>laser_frame</frame_name>

File: description/robot.urdf.xacro (robot description, xacro)
@@ -1,7 +1,15 @@
 <?xml version="1.0"?>
 <robot xmlns:xacro="http://www.ros.org/wiki/xacro"  name="robot">
+    <xacro:arg name="use_ros2_control" default="true"/>
     <xacro:include filename="robot_core.xacro" />
-    <xacro:include filename="gazebo_control.xacro" />
+    <xacro:if value="$(arg use_ros2_control)">
+        <xacro:include filename="ros2_control.xacro" />
+    </xacro:if>
+    <xacro:unless value="$(arg use_ros2_control)">
+        <xacro:include filename="gazebo_control.xacro" />
+    </xacro:unless>
     <xacro:include filename="lidar.xacro" />
     <xacro:include filename="camera.xacro" />
+    <!-- <xacro:include filename="depth_camera.xacro" /> -->
+    <!-- <xacro:include filename="face.xacro" /> -->
 </robot>

File: description/robot_core.xacro (robot description, xacro)
@@ -64,5 +64,5 @@
        <collision>
            <geometry>
-               <cylinder radius= "0.05" length="0.04"/>
+               <sphere radius= "0.05" />
            </geometry>
            <material name="blue"/>
@@ -91,5 +91,5 @@
        <collision>
            <geometry>
-               <cylinder radius= "0.05" length="0.04"/>
+               <sphere radius= "0.05" />
            </geometry>
            <material name="blue"/>
@@ -118,5 +118,5 @@
        <collision>
            <geometry>
-               <cylinder radius= "0.05" length="0.04"/>
+               <sphere radius= "0.05" />
            </geometry>
            <material name="blue"/>
@@ -145,5 +145,5 @@
       <collision>
            <geometry>
-               <cylinder radius= "0.05" length="0.04"/>
+               <sphere radius= "0.05" />
            </geometry>
            <material name="blue"/>
