Commit message: realrobot

File: description/lidar.xacro (robot description, xacro)
@@ -4,5 +4,5 @@
         <parent link="chassis"/>
         <child link="laser_frame"/>
-        <origin xyz="0.025 0 0.1" rpy="0 0 0"/>
+        <origin xyz="0.0 0 0.1" rpy="0 0 0"/>
     </joint>
     <link name="laser_frame">

File: description/robot.urdf.xacro (robot description, xacro)
@@ -3,6 +3,7 @@
     <xacro:include filename="robot_core.xacro" />
     <xacro:include filename="lidar.xacro" />
-    <!-- <xacro:include filename="ros2_control.xacro" /> -->
-    <xacro:include filename="imu.xacro" />
-    <xacro:include filename="gazebo_control.xacro" />
+    <xacro:include filename="ros2_control.xacro" />
+    <!-- <xacro:include filename="imu.xacro" /> -->
+    <!-- <xacro:include filename="gazebo_control.xacro" /> -->
+    <xacro:include filename="arm.xacro" />
 </robot>

File: description/robot_core.xacro (robot description, xacro)
@@ -2,7 +2,7 @@
 <robot xmlns:xacro="http://www.ros.org/wiki/xacro" >
     <xacro:include filename="inertial_macros.xacro"/>
-    <xacro:property name="chassis_length" value="0.23"/>
-    <xacro:property name="chassis_width" value="0.23"/>
-    <xacro:property name="chassis_height" value="0.1085"/>
+    <xacro:property name="chassis_length" value="0.15"/>
+    <xacro:property name="chassis_width" value="0.15"/>
+    <xacro:property name="chassis_height" value="0.13"/>
     <xacro:property name="chassis_mass" value="1.0"/>
     <xacro:property name="wheel_radius" value="0.033"/>
@@ -10,9 +10,9 @@
     <xacro:property name="wheel_mass" value="0.05"/>
     <xacro:property name="wheel_offset_x" value="0.045"/>
-    <xacro:property name="wheel_offset_y" value="0.1265"/>
-    <xacro:property name="wheel_offset_z" value="0.03275"/>
+    <xacro:property name="wheel_offset_y" value="0.10"/>
+    <xacro:property name="wheel_offset_z" value="0.04"/>
     <!-- <xacro:property name="caster_wheel_radius" value="${0.01*1}"/> -->
     <xacro:property name="caster_wheel_mass" value="0.01"/>
-    <xacro:property name="caster_wheel_offset_x" value="0.075"/>
+    <xacro:property name="caster_wheel_offset_x" value="0.06"/>
     <!-- <xacro:property name="caster_wheel_offset_y" value="0.1265"/> -->
     <!-- <xacro:property name="caster_wheel_offset_z" value="0.05475"/> -->

File: description/ros2_control.xacro (robot description, xacro)
@@ -1,5 +1,34 @@
 <?xml version="1.0"?>
 <robot xmlns:xacro="http://www.ros.org/wiki/xacro">
-<ros2_control name="GazeboSystem" type="system">
+    <ros2_control name="RealRobot" type="system">
+        <hardware>
+            <plugin>diffdrive_arduino/DiffDriveArduinoHardware</plugin>
+            <param name="left_wheel_name">left_wheel_joint</param>
+            <param name="right_wheel_name">right_wheel_joint</param>
+            <param name="loop_rate">50</param>
+            <param name="device">/dev/ttyUSB0</param>
+            <param name="baud_rate">57600</param>
+            <param name="timeout_ms">1000</param>
+            <param name="enc_counts_per_rev">5800</param>
+        </hardware>
+        <!-- Note everything below here is the same as the Gazebo one -->
+        <joint name="left_wheel_joint">
+            <command_interface name="velocity">
+                <param name="min">-10</param>
+                <param name="max">10</param>
+            </command_interface>
+            <state_interface name="position"/>
+            <state_interface name="velocity"/>
+        </joint>
+        <joint name="right_wheel_joint">
+            <command_interface name="velocity">
+                <param name="min">-10</param>
+                <param name="max">10</param>
+            </command_interface>
+            <state_interface name="position"/>
+            <state_interface name="velocity"/>
+        </joint>
+    </ros2_control>
+<!-- <ros2_control name="GazeboSystem" type="system">
   <hardware>
         <plugin>gazebo_ros2_control/GazeboSystem</plugin>
@@ -21,5 +50,5 @@
                 <state_interface name="position"/>
         </joint>
-</ros2_control>
+</ros2_control>   -->
     <gazebo>
         <plugin name="gazebo_ros2_control" filename="libgazebo_ros2_control.so">
