Commit message: update new model

File: description/arm.xacro (robot description, xacro)
@@ -4,26 +4,41 @@
         <parent link="chassis"/>
         <child link="arm_frame"/>
-        <origin xyz="0.0 0 0.075" rpy="0 0 0"/>
+        <origin xyz="-0.03 0.0 0.075" rpy="0 0 0"/>
     </joint>
     <link name="arm_frame">
         <visual>
+            <origin xyz="0 0 0.05"/>
             <geometry>
                 <box size="0.02 0.02 0.1"/>
             </geometry>
-            <material name="black"/>
+            <material name="brown"/>
         </visual>
         <visual>
-            <origin xyz="0 0 0"/>
+            <origin xyz="0.13 0 0.10"/>
             <geometry>
-                <box size="0.26 0.02 0.02"/>
+                <box size="0.28 0.02 0.02"/>
             </geometry>
-            <material name="black"/>
+            <material name="brown"/>
+        </visual>
+        <visual>
+            <origin xyz="0.28 0 0.10"/>
+            <geometry>
+                <box size="0.02 0.20 0.02"/>
+            </geometry>
+            <material name="brown"/>
         </visual>
         <collision>
-            <origin xyz="0 0 0"/>
+            <origin xyz="0.13 0 10"/>
             <geometry>
-                <box size="0.26 0.02 0.02"/>
+                <box size="0.28 0.02 0.02"/>
             </geometry>
-            <material name="black"/>
+            <material name="brown"/>
+        </collision>
+        <collision>
+            <origin xyz="0.28 0 0.10"/>
+            <geometry>
+                <box size="0.02 0.20 0.02"/>
+            </geometry>
+            <material name="brown"/>
         </collision>
         <!-- <xacro:inertial_box mass="0.03" x="${chassis_length}" y="${chassis_width}" z="${chassis_height}">

File: description/robot.urdf.xacro (robot description, xacro)
@@ -6,4 +6,4 @@
     <!-- <xacro:include filename="imu.xacro" /> -->
     <!-- <xacro:include filename="gazebo_control.xacro" /> -->
-    <xacro:include filename="arm.xacro" />
+    <!-- <xacro:include filename="arm.xacro" /> -->
 </robot>

File: description/robot_core.xacro (robot description, xacro)
@@ -4,11 +4,11 @@
     <xacro:property name="chassis_length" value="0.15"/>
     <xacro:property name="chassis_width" value="0.15"/>
-    <xacro:property name="chassis_height" value="0.13"/>
+    <xacro:property name="chassis_height" value="0.12"/>
     <xacro:property name="chassis_mass" value="1.0"/>
-    <xacro:property name="wheel_radius" value="0.033"/>
+    <xacro:property name="wheel_radius" value="0.034"/>
     <xacro:property name="wheel_thickness" value="0.026"/>
     <xacro:property name="wheel_mass" value="0.05"/>
-    <xacro:property name="wheel_offset_x" value="0.045"/>
-    <xacro:property name="wheel_offset_y" value="0.10"/>
+    <xacro:property name="wheel_offset_x" value="0.04"/>
+    <xacro:property name="wheel_offset_y" value="0.0975"/>
     <xacro:property name="wheel_offset_z" value="0.04"/>
     <!-- <xacro:property name="caster_wheel_radius" value="${0.01*1}"/> -->
@@ -31,4 +31,10 @@
     <material name="red">
         <color rgba="1 0 0 1"/>
+    </material>
+    <material name="green">
+        <color rgba="0 1 0 1"/>
+    </material>
+    <material name="brown">
+        <color rgba="0.6 0.3 0.1 1"/>
     </material>
     <!-- BASE LINK -->

File: description/ros2_control.xacro (robot description, xacro)
@@ -10,11 +10,11 @@
             <param name="baud_rate">57600</param>
             <param name="timeout_ms">1000</param>
-            <param name="enc_counts_per_rev">5800</param>
+            <param name="enc_counts_per_rev">5767</param>
         </hardware>
         <!-- Note everything below here is the same as the Gazebo one -->
         <joint name="left_wheel_joint">
             <command_interface name="velocity">
-                <param name="min">-10</param>
-                <param name="max">10</param>
+                <param name="min">-5</param>
+                <param name="max">5</param>
             </command_interface>
             <state_interface name="position"/>
@@ -23,6 +23,6 @@
         <joint name="right_wheel_joint">
             <command_interface name="velocity">
-                <param name="min">-10</param>
-                <param name="max">10</param>
+                <param name="min">-5</param>
+                <param name="max">5</param>
             </command_interface>
             <state_interface name="position"/>
